File: PCB/board1.sch (EAGLE design)
At the start: 36 parts, among them J1 5.5x2.1mm Barrel, U1 MAX3485CSA, U2 SI7021, U3 PHOTON, U4 LMR14020

Commit message: Added solidworks files
Parts:
- renumbered U$2 to FID2, U$3 to FID1
Changed lines of the file:
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@@
 <?xml version="1.0" encoding="utf-8"?>
 <!DOCTYPE eagle SYSTEM "eagle.dtd">
-<eagle version="8.6.0">
+<eagle version="9.0.0">
 <drawing>
 <settings>
@@
 <part name="C1" library="rcl" library_urn="urn:adsk.eagle:library:334" deviceset="C-US" device="C0805" package3d_urn="urn:adsk.eagle:package:23617/1" value="100nF"/>
 <part name="R1" library="rcl" library_urn="urn:adsk.eagle:library:334" deviceset="R-US_" device="R0805" package3d_urn="urn:adsk.eagle:package:23553/1" value="4.7k"/>
-<part name="U$2" library="adafruit" library_urn="urn:adsk.eagle:library:420" deviceset="FIDUCIAL" device=""/>
-<part name="U$3" library="adafruit" library_urn="urn:adsk.eagle:library:420" deviceset="FIDUCIAL" device=""/>
+<part name="FID2" library="adafruit" library_urn="urn:adsk.eagle:library:420" deviceset="FIDUCIAL" device=""/>
+<part name="FID1" library="adafruit" library_urn="urn:adsk.eagle:library:420" deviceset="FIDUCIAL" device=""/>
 <part name="D1" library="standardparts" deviceset="LED" device=".0805"/>
 <part name="POWER1" library="SparkFun-Connectors" deviceset="CONN_02" device="5MM"/>
@@
 <instance part="C1" gate="G$1" x="223.52" y="17.78"/>
 <instance part="R1" gate="G$1" x="180.34" y="76.2" rot="R180"/>
-<instance part="U$2" gate="G$1" x="182.88" y="53.34"/>
-<instance part="U$3" gate="G$1" x="172.72" y="53.34"/>
+<instance part="FID2" gate="G$1" x="182.88" y="53.34"/>
+<instance part="FID1" gate="G$1" x="172.72" y="53.34"/>
 <instance part="D1" gate="G$1" x="190.5" y="76.2"/>
 <instance part="POWER1" gate="G$1" x="10.16" y="60.96"/>
